Commit message: 该修改作为重新开始的证明

File: src/usv_sim_full/description/urdf/wamv_base.urdf.xacro (robot description, xacro)
@@ -3,4 +3,9 @@
   <!-- Required arg for melodic and kinetic... -->
   <xacro:arg name="namespace" default="wamv"/>
+  <!-- Allow overriding the base mass and inertial tensor from top-level xacro args -->
+  <xacro:arg name="mass" default="1900.0"/>
+  <xacro:arg name="ixx" default="1200"/>
+  <xacro:arg name="iyy" default="4000"/>
+  <xacro:arg name="izz" default="4500"/>
   <xacro:property name="namespace" value="$(arg namespace)" scope="global" />
   <!-- Macro for creating the main collisions as simple shapes. -->
@@ -105,9 +110,9 @@
     </collision>
     <inertial>
-      <!-- From WAM-V spec sheet -->
-      <mass value="1900.0"/>
+      <!-- Mass and inertia can be overridden via top-level xacro args -->
+      <mass value="$(arg mass)"/>
       <origin xyz="0 0 -0.2" rpy="0 0 0"/>
-      <!-- 惯性张量根据 1.9 吨、5m长、2.5m宽估算 -->
-      <inertia ixx="1200" ixy="0" ixz="0" iyy="4000" iyz="0" izz="4500"/>
+      <!-- Inertia tensor (diagonal) -->
+      <inertia ixx="$(arg ixx)" ixy="0" ixz="0" iyy="$(arg iyy)" iyz="0" izz="$(arg izz)"/>
     </inertial>
   </link>

File: src/usv_sim_full/templates/wamv_base.urdf.xacro (robot description, xacro)
@@ -110,8 +110,8 @@
     </collision>
     <inertial>
-      <!-- Mass and inertia read from args (with defaults defined at the top) -->
+      <!-- From WAM-V spec sheet -->
       <mass value="$(arg mass)"/>
       <origin xyz="0 0 -0.2" rpy="0 0 0"/>
-      <!-- Inertia tensor (diagonal) -->
+      <!-- 惯性张量根据 1.9 吨、5m长、2.5m宽估算 -->
       <inertia ixx="$(arg ixx)" ixy="0" ixz="0" iyy="$(arg iyy)" iyz="0" izz="$(arg izz)"/>
     </inertial>

File: src/usv_sim_full/templates/wamv_no_battery.urdf.xacro (robot description, xacro)
@@ -41,4 +41,13 @@
   <xacro:arg name="nR" default="800.0"/>
   <xacro:arg name="nRR" default="800.0"/>
+  <!-- Mass / inertia overrides (top-level args exposed as global properties so included files see them) -->
+  <xacro:arg name="mass" default="1900.0"/>
+  <xacro:arg name="ixx" default="1200"/>
+  <xacro:arg name="iyy" default="4000"/>
+  <xacro:arg name="izz" default="4500"/>
+  <xacro:property name="mass" value="$(arg mass)" scope="global" />
+  <xacro:property name="ixx" value="$(arg ixx)" scope="global" />
+  <xacro:property name="iyy" value="$(arg iyy)" scope="global" />
+  <xacro:property name="izz" value="$(arg izz)" scope="global" />
   <xacro:property name="thruster_namespace" value="$(arg thruster_namespace)" scope="global" />
   <xacro:property name="camera_namespace" value="$(arg camera_namespace)" scope="global" />
@@ -54,6 +63,10 @@
   <xacro:arg name="thruster_xacro_file" default = ""/>
   <!-- === WAM-V平台 === -->
-  <xacro:arg name="macros_file" default="$(find wamv_gazebo)/urdf/macros.xacro"/>
-  <xacro:include filename="$(find wamv_gazebo)/urdf/wamv_gazebo.xacro"/>
+  <!-- Use a local override of wamv_gazebo to avoid automatically injecting
+    the upstream dynamics plugin. The override includes sensor macros
+    but does NOT call the usv_dynamics_gazebo macro, allowing this
+    file to provide custom gazebo plugin blocks below. -->
+  <xacro:arg name="macros_file" default="$(find usv_sim_full)/templates/macros_without_dynamics.xacro"/>
+  <xacro:include filename="$(find usv_sim_full)/templates/wamv_gazebo_override.xacro"/>
   <!-- === 电池已移除 === -->
   <!-- === 推进器 === -->
@@ -93,23 +106,5 @@
   </gazebo>
   <!-- === TF变换 === -->
-  <!-- 发布机器人状态信息 -->
-  <gazebo>
-    <plugin filename="libgz-sim-pose-publisher-system.so"
-      name="gz::sim::systems::PosePublisher">
-      <publish_link_pose>false</publish_link_pose>
-      <publish_sensor_pose>true</publish_sensor_pose>
-      <publish_collision_pose>false</publish_collision_pose>
-      <publish_visual_pose>false</publish_visual_pose>
-      <publish_nested_model_pose>false</publish_nested_model_pose>
-      <publish_model_pose>false</publish_model_pose>
-      <use_pose_vector_msg>true</use_pose_vector_msg>
-      <static_publisher>false</static_publisher>
-      <static_update_frequency>1</static_update_frequency>
-    </plugin>
-    <plugin
-      filename="gz-sim-joint-state-publisher-system"
-      name="gz::sim::systems::JointStatePublisher">
-    </plugin>
-  </gazebo>
+  <!-- (removed malformed/duplicated inertial and plugin block; inertial is defined in description/urdf/wamv_base.urdf.xacro) -->
   <!-- === 传感器 === -->
   <!-- 如果提供了传感器yaml文件，则使用它 -->
@@ -178,52 +173,11 @@
   </xacro:if>
   <!-- === 水动力学插件 - 使用配置参数 === -->
-  <gazebo>
-    <!-- 左船体 -->
-    <plugin filename="libSurface.so" name="vrx::Surface">
-      <link_name>$(arg namespace)/base_link</link_name>
-      <hull_length>$(arg hull_length)</hull_length>
-      <hull_radius>$(arg hull_radius)</hull_radius>
-      <fluid_level>$(arg fluid_level)</fluid_level>
-      <points>
-        <point>0.6 1.03 0</point>
-        <point>-1.4 1.03 0</point>
-      </points>
-      <wavefield>
-        <topic>/vrx/wavefield/parameters</topic>
-      </wavefield>
-    </plugin>
-    <!-- 右船体 -->
-    <plugin filename="libSurface.so" name="vrx::Surface">
-      <link_name>$(arg namespace)/base_link</link_name>
-      <hull_length>$(arg hull_length)</hull_length>
-      <hull_radius>$(arg hull_radius)</hull_radius>
-      <fluid_level>$(arg fluid_level)</fluid_level>
-      <points>
-        <point>0.6 -1.03 0</point>
-        <point>-1.4 -1.03 0</point>
-      </points>
-      <wavefield>
-        <topic>/vrx/wavefield/parameters</topic>
-      </wavefield>
-    </plugin>
-    <plugin filename="libSimpleHydrodynamics.so" name="vrx::SimpleHydrodynamics">
-      <link_name>$(arg namespace)/base_link</link_name>
-      <!-- 附加质量 -->
-      <xDotU>$(arg xDotU)</xDotU>
-      <yDotV>$(arg yDotV)</yDotV>
-      <nDotR>$(arg nDotR)</nDotR>
-      <!-- 线性和二次阻力 -->
-      <xU>$(arg xU)</xU>
-      <xUU>$(arg xUU)</xUU>
-      <yV>$(arg yV)</yV>
-      <yVV>$(arg yVV)</yVV>
-      <zW>$(arg zW)</zW>
-      <kP>$(arg kP)</kP>
-      <kPP>$(arg kPP)</kPP>
-      <mQ>$(arg mQ)</mQ>
-      <mQQ>$(arg mQQ)</mQQ>
-      <nR>$(arg nR)</nR>
-      <nRR>$(arg nRR)</nRR>
-    </plugin>
-  </gazebo>
+  <!-- 使用本地参数化 dynamics 宏，将顶层 args 传递给插件 -->
+  <xacro:include filename="$(find usv_sim_full)/templates/wamv_gazebo_dynamics_param.xacro"/>
+  <xacro:usv_dynamics_gazebo name="wamv_dynamics_plugin"
+    hull_length="$(arg hull_length)" hull_radius="$(arg hull_radius)" fluid_level="$(arg fluid_level)"
+    xDotU="$(arg xDotU)" yDotV="$(arg yDotV)" nDotR="$(arg nDotR)"
+    xU="$(arg xU)" xUU="$(arg xUU)" yV="$(arg yV)" yVV="$(arg yVV)"
+    zW="$(arg zW)" kP="$(arg kP)" kPP="$(arg kPP)" mQ="$(arg mQ)" mQQ="$(arg mQQ)"
+    nR="$(arg nR)" nRR="$(arg nRR)"/>
 </robot>
