Commit message: fix: publish zero thrust unconditionally on cmd timeout
- cmd_vel_to_thruster.py: remove _cmd_active guard from cmd_timeout
  branch so zero thrust is always written to Gazebo on first startup,
  preventing uncontrolled coasting
- wamv_gazebo_thruster_config.xacro: raise max_velocity_mps from
  7.72 to 15.0 m/s, increasing Gazebo max_thrust_cmd ceiling to
  ~8530 N per thruster

File: vrx/vrx_urdf/wamv_gazebo/urdf/thruster_layouts/wamv_gazebo_thruster_config.xacro (robot description, xacro)
@@ -5,5 +5,5 @@
     <xacro:property name="x_uu" value="72.4" />
     <xacro:property name="x_u" value="51.3" />
-    <xacro:property name="max_velocity_mps" value="7.71667" />
+    <xacro:property name="max_velocity_mps" value="15.0" />
     <plugin
       filename="gz-sim-thruster-system"
