Commit message: Revert "feat(毫米波): 对齐 MmwaveTarget 聚类输出与三视觉 bringup 配置 (#2)"
This reverts commit 37ccd46c0b1e462bda07bf102a2ed798a350cb4c.

File: vrx/vrx_urdf/wamv_gazebo/urdf/thruster_layouts/wamv_gazebo_thruster_config.xacro (robot description, xacro)
@@ -5,5 +5,5 @@
     <xacro:property name="x_uu" value="72.4" />
     <xacro:property name="x_u" value="51.3" />
-    <xacro:property name="max_velocity_mps" value="15.0" />
+    <xacro:property name="max_velocity_mps" value="7.71667" />
     <plugin
       filename="gz-sim-thruster-system"
