Commit message: chore(file)调整usv_sim_full文件目录，移除重复文件，修改对应加载逻辑

File: usv_sim_full/description/urdf/cpu_cases.xacro (robot description, xacro)
@@ -6,5 +6,5 @@
       <origin xyz="0.073 0 -1.53" rpy="0 0 0"/>
       <geometry>
-        <mesh filename="package://usv_sim_full/description/models/cpu_cases/mesh/cpu_cases.dae"/>
+        <mesh filename="package://vrx_gz/models/cpu_cases/mesh/cpu_cases.dae"/>
       </geometry>
     </visual>

File: usv_sim_full/description/urdf/custom_thrusters.xacro (robot description, xacro)
@@ -15,6 +15,26 @@
     prefix="right"
     position="$(arg thruster_pos_x) $(arg thruster_pos_y_right) $(arg thruster_pos_z)" />
-  <xacro:include filename="$(find wamv_gazebo)/urdf/thruster_layouts/wamv_gazebo_thruster_config.xacro" />
-  <xacro:wamv_gazebo_thruster_config name="left" />
-  <xacro:wamv_gazebo_thruster_config name="right" />
+  <xacro:macro name="thruster_plugin" params="name">
+    <gazebo>
+      <plugin filename="gz-sim-thruster-system" name="gz::sim::systems::Thruster">
+        <joint_name>${namespace}/${name}_engine_propeller_joint</joint_name>
+        <thrust_coefficient>0.004422</thrust_coefficient>
+        <fluid_density>1000</fluid_density>
+        <propeller_diameter>0.2</propeller_diameter>
+        <velocity_control>true</velocity_control>
+        <max_thrust_cmd>853.95</max_thrust_cmd>
+        <namespace>${namespace}</namespace>
+        <topic>thrusters/${name}/thrust</topic>
+        <name>${name}</name>
+      </plugin>
+      <plugin filename="gz-sim-joint-position-controller-system" name="gz::sim::systems::JointPositionController">
+        <joint_name>${namespace}/${name}_chassis_engine_joint</joint_name>
+        <use_velocity_commands>true</use_velocity_commands>
+        <topic>${namespace}/thrusters/${name}/pos</topic>
+        <name>${name}</name>
+      </plugin>
+    </gazebo>
+  </xacro:macro>
+  <xacro:thruster_plugin name="left" />
+  <xacro:thruster_plugin name="right" />
 </robot>

File: usv_sim_full/description/urdf/hull_macro.xacro (robot description, xacro)
@@ -6,5 +6,5 @@
     mass:=180.0
     ixx:=100.0 iyy:=100.0 izz:=200.0
-    visual_mesh:=package://usv_sim_full/description/models/WAM-V-Base/mesh/WAM-V-Base.dae
+    visual_mesh:=package://vrx_gz/models/body-Base/mesh/M5_body.dae
     xyz:='0 0 0'
     rpy:='0 0 0'">

File: usv_sim_full/description/urdf/mb_marker_buoy.urdf.xacro (robot description, xacro)
@@ -9,5 +9,5 @@
       <origin xyz="0 0 0" rpy="1.57079 0 0"/>
       <geometry>
-        <mesh filename="package://usv_sim_full/description/models/mb_marker_buoy/meshes/mb_marker_buoy.dae"/>
+        <mesh filename="package://vrx_gz/models/mb_marker_buoy/meshes/mb_marker_buoy.dae"/>
       </geometry>
     </visual>

File: usv_sim_full/description/urdf/sensor_macros.xacro (robot description, xacro)
@@ -156,5 +156,5 @@
     <link name="${name}_mount_link">
       <inertial><mass value="0.30"/><inertia ixx="0.002" ixy="0" ixz="0" iyy="0.002" iyz="0" izz="0.002"/></inertial>
-      <visual><geometry><mesh filename="package://usv_sim_full/description/models/px4_gimbal/meshes/cgo3_mount_remeshed_v1.stl" scale="0.001 0.001 0.001"/></geometry><material name="gray"><color rgba="0.25 0.25 0.25 1"/></material></visual>
+      <visual><geometry><mesh filename="package://vrx_gz/models/px4_gimbal/meshes/cgo3_mount_remeshed_v1.stl" scale="0.001 0.001 0.001"/></geometry><material name="gray"><color rgba="0.25 0.25 0.25 1"/></material></visual>
       <collision><geometry><cylinder radius="0.09" length="0.05"/></geometry></collision>
     </link>
@@ -164,5 +164,5 @@
     <link name="${name}_yaw_link">
       <inertial><mass value="0.20"/><inertia ixx="0.001" ixy="0" ixz="0" iyy="0.001" iyz="0" izz="0.001"/></inertial>
-      <visual><geometry><mesh filename="package://usv_sim_full/description/models/px4_gimbal/meshes/cgo3_vertical_arm_remeshed_v1.stl" scale="0.001 0.001 0.001"/></geometry><material name="dark_gray"><color rgba="0.15 0.15 0.15 1"/></material></visual>
+      <visual><geometry><mesh filename="package://vrx_gz/models/px4_gimbal/meshes/cgo3_vertical_arm_remeshed_v1.stl" scale="0.001 0.001 0.001"/></geometry><material name="dark_gray"><color rgba="0.15 0.15 0.15 1"/></material></visual>
       <collision><geometry><cylinder radius="0.06" length="0.07"/></geometry></collision>
     </link>
@@ -173,5 +173,5 @@
     <link name="${name}_roll_link">
       <inertial><mass value="0.15"/><inertia ixx="0.0005" ixy="0" ixz="0" iyy="0.0005" iyz="0" izz="0.0005"/></inertial>
-      <visual><geometry><mesh filename="package://usv_sim_full/description/models/px4_gimbal/meshes/cgo3_horizontal_arm_remeshed_v1.stl" scale="0.001 0.001 0.001"/></geometry><material name="black"><color rgba="0.08 0.08 0.08 1"/></material></visual>
+      <visual><geometry><mesh filename="package://vrx_gz/models/px4_gimbal/meshes/cgo3_horizontal_arm_remeshed_v1.stl" scale="0.001 0.001 0.001"/></geometry><material name="black"><color rgba="0.08 0.08 0.08 1"/></material></visual>
       <collision><geometry><box size="0.12 0.05 0.05"/></geometry></collision>
     </link>
@@ -193,5 +193,5 @@
     <link name="${name}_camera_link">
       <inertial><mass value="0.15"/><inertia ixx="0.0004" ixy="0" ixz="0" iyy="0.0004" iyz="0" izz="0.0004"/></inertial>
-      <visual><geometry><mesh filename="package://usv_sim_full/description/models/px4_gimbal/meshes/cgo3_camera_remeshed_v1.stl" scale="0.001 0.001 0.001"/></geometry><material name="camera_black"><color rgba="0.02 0.02 0.02 1"/></material></visual>
+      <visual><geometry><mesh filename="package://vrx_gz/models/px4_gimbal/meshes/cgo3_camera_remeshed_v1.stl" scale="0.001 0.001 0.001"/></geometry><material name="camera_black"><color rgba="0.02 0.02 0.02 1"/></material></visual>
       <collision><geometry><box size="0.10 0.08 0.06"/></geometry></collision>
     </link>

File: usv_sim_full/description/urdf/thrusters/engine.xacro (robot description, xacro)
@@ -6,5 +6,5 @@
       <visual>
         <geometry>
-          <mesh filename="package://usv_sim_full/description/models/engine/mesh/engine.dae"/>
+          <mesh filename="package://vrx_gz/models/engine/mesh/engine.dae"/>
         </geometry>
       </visual>
@@ -29,5 +29,5 @@
       <visual>
         <geometry>
-          <mesh filename="package://usv_sim_full/description/models/propeller/mesh/propeller.dae"/>
+          <mesh filename="package://vrx_gz/models/propeller/mesh/propeller.dae"/>
         </geometry>
       </visual>

File: usv_sim_full/description/urdf/usv_gazebo.xacro (robot description, xacro)
@@ -1,6 +1,4 @@
 <?xml version="1.0"?>
 <robot xmlns:xacro="http://ros.org/wiki/xacro">
-  <!-- Include macros for dynamics plugins -->
-  <xacro:include filename="$(arg macros_file)" />
   <!-- Macro to create a USV with dynamics plugins and a customizeable thruster layout -->
   <xacro:macro name="usv_gazebo" params="thruster_layout">

File: usv_sim_full/description/urdf/wamv_base.urdf.xacro (robot description, xacro)
@@ -8,5 +8,5 @@
   <xacro:arg name="iyy" default="4000"/>
   <xacro:arg name="izz" default="4500"/>
-  <xacro:arg name="visual_mesh" default="package://usv_sim_full/description/models/WAM-V-Base/mesh/M5_body.dae"/>
+  <xacro:arg name="visual_mesh" default="package://vrx_gz/models/body-Base/mesh/M5_body.dae"/>
   <xacro:property name="namespace" value="$(arg namespace)" scope="global" />
   <!-- Macro for creating the main collisions as simple shapes. -->
@@ -98,5 +98,4 @@
       </geometry>
     </visual>
-    <!-- <mesh filename="package://usv_sim_full/description/models/WAM-V-Base/mesh/WAM-V-Base.dae"/> -->
 <!-- src/my_wamv/blade_R.dae -->
     <!-- Left base collisions -->

File: usv_sim_full/description/urdf/wamv_no_battery.urdf.xacro (robot description, xacro)
@@ -22,6 +22,6 @@
   <!-- 注意：这只用于一些没有正确使用robotNamespace参数的传感器 -->
   <xacro:arg name="namespace" default="wamv"/>
-  <!-- VRX 场景：将船系在 platform 上；多船自航仿真应关闭，避免争抢同一 child_model 导致只成功 spawn 一艘 -->
-  <xacro:arg name="enable_detachable_joint" default="true"/>
+  <!-- 当前场景不包含 VRX platform；仅在显式请求时才启用系泊关节。 -->
+  <xacro:arg name="enable_detachable_joint" default="false"/>
   <xacro:arg name="has_extra_sensors" default="false"/>
   <xacro:arg name="extra_sensors" default=""/>
@@ -57,5 +57,4 @@
   <xacro:arg name="thruster_xacro_file" default = ""/>
   <!-- === WAM-V平台 === -->
-  <xacro:arg name="macros_file" default="$(find wamv_gazebo)/urdf/macros.xacro"/>
   <xacro:include filename="$(find usv_sim_full)/description/urdf/usv_gazebo.xacro"/>
   <!-- === 电池已移除 === -->
@@ -68,16 +67,4 @@
   <xacro:unless value="$(arg yaml_thruster_generation)">
     <xacro:property name="thruster_conf" value="$(arg thruster_config)"/>
-    <!-- 默认WAM-V，带有两个后部推进器 -->
-    <xacro:if value="${thruster_conf == 'H'}">
-       <xacro:usv_gazebo thruster_layout="$(find wamv_gazebo)/urdf/thruster_layouts/wamv_aft_thrusters.xacro"/>
-    </xacro:if>
-    <!-- "T"型推进器配置的WAMV -->
-    <xacro:if value="${thruster_conf == 'T'}">
-      <xacro:usv_gazebo thruster_layout="$(find wamv_gazebo)/urdf/thruster_layouts/wamv_t_thrusters.xacro"/>
-    </xacro:if>
-    <!-- "X"型推进器配置的WAMV -->
-    <xacro:if value="${thruster_conf == 'X'}">
-      <xacro:usv_gazebo thruster_layout="$(find wamv_gazebo)/urdf/thruster_layouts/wamv_x_thrusters.xacro"/>
-    </xacro:if>
     <!-- 自定义推进器配置 -->
     <xacro:if value="${thruster_conf == 'CUSTOM'}">
@@ -127,56 +114,14 @@
     <xacro:cpu_cases position="-0.15 0 1.53" orientation="0 0 0"/>
   </xacro:if>
-  <!-- 否则，根据启用变量添加传感器 -->
-  <xacro:unless value="$(arg yaml_component_generation)">
-    <!-- 添加前摄像头 -->
-    <xacro:if value="$(arg camera_enabled)">
-      <xacro:wamv_camera name="front_camera" y="0.3" x="0.75" P="${radians(15)}" />
-    </xacro:if>
-    <!-- 添加模拟GPS -->
-    <xacro:if value="$(arg gps_enabled)">
-      <xacro:wamv_gps name="gps_wamv" x="-0.85" />
-    </xacro:if>
-    <!-- 添加模拟IMU -->
-    <xacro:if value="$(arg imu_enabled)">
-      <xacro:wamv_imu name="imu_wamv" y="-0.2" />
-    </xacro:if>
-    <!-- 添加3D激光雷达 -->
-    <xacro:if value="$(arg lidar_enabled)">
-      <xacro:lidar name="lidar_wamv" y="-0.3" type="16_beam"/>
-    </xacro:if>
-    <!-- 添加P3D真实值 -->
-    <xacro:if value="$(arg ground_truth_enabled)">
-      <xacro:wamv_p3d name="p3d_wamv"/>
-    </xacro:if>
-    <!-- 添加声学信标 -->
-    <xacro:if value="$(arg pinger_enabled)">
-      <xacro:wamv_pinger sensor_name="receiver" position="-528 191 -2.0" />
-    </xacro:if>
-    <!-- 添加球发射器（默认俯仰角：~-60度） -->
-    <xacro:if value="$(arg ball_shooter_enabled)">
-      <xacro:wamv_ball_shooter name="ball_shooter" x="0.54" y="0.30" z="1.296" pitch="-1.04"/>
-    </xacro:if>
-    <!-- ==== VRX传感器配置 ==== -->
-    <xacro:if value="$(arg vrx_sensors_enabled)">
-      <!-- 添加CPU外壳 -->
-      <xacro:include filename="$(find usv_sim_full)/description/urdf/cpu_cases.xacro" />
-      <xacro:cpu_cases position="-0.15 0 1.53" orientation="0 0 0"/>
-      <!-- 添加一个立体相机对 -->
-      <xacro:wamv_camera name="front_left_camera" y="0.1" x="0.75" P="${radians(15)}" />
-      <xacro:wamv_camera name="front_right_camera" y="-0.1" x="0.75" P="${radians(15)}" />
-      <!-- 添加一个朝右的相机 -->
-      <xacro:wamv_camera name="middle_right_camera" y="-0.45" P="${radians(15)}" Y="${radians(-90)}" post_Y="${radians(-90)}" />
-      <!-- 添加模拟GPS -->
-      <xacro:wamv_gps name="gps_wamv" x="-0.85" />
-      <!-- 添加模拟IMU -->
-      <xacro:wamv_imu name="imu_wamv" y="-0.2" />
-      <!-- 添加3D激光雷达 -->
-      <xacro:lidar name="lidar_wamv" type="16_beam"/>
-      <!-- 添加声学信标 -->
-      <xacro:wamv_pinger sensor_name="receiver" position="-528 191 -2.0" />
-      <!-- 添加球发射器（默认俯仰角：~-60度） -->
-      <xacro:wamv_ball_shooter name="ball_shooter" x="0.54" y="0.30" z="1.296" pitch="-1.04"/>
-    </xacro:if>
-  </xacro:unless>
+  <xacro:if value="$(arg ground_truth_enabled)">
+    <gazebo>
+      <plugin filename="gz-sim-odometry-publisher-system" name="gz::sim::systems::OdometryPublisher">
+        <dimensions>3</dimensions>
+        <odom_publish_frequency>30.0</odom_publish_frequency>
+        <odom_frame>$(arg namespace)/odom</odom_frame>
+        <robot_base_frame>$(arg namespace)/base_link</robot_base_frame>
+      </plugin>
+    </gazebo>
+  </xacro:if>
   <!-- === 包含额外传感器配置 === -->
   <xacro:if value="$(arg has_extra_sensors)">
